File: hardware/badge-esp32-s3/leds.kicad_sch (KiCad schematic)
At the start: 29 parts

Commit message: minibadge_fix?
Parts:
- AL1, AL2, AL3, AL4, AL5, AL6, AL7: JLC_3DModel_Q (none) -> c6c295f7aed14366abe0e80218141640; JLC_3D_Size (none) -> 2.2 2.2; LCSC Part (none) -> C22371528; Supplier Part C22371528 -> (none)
- AL10, AL11, AL12, AL13, AL14, AL15, AL16, AL17, AL18, AL19, AL20, AL21, AL22, AL23, AL8, AL9: JLC_3DModel_Q (none) -> c6c295f7aed14366abe0e80218141640; JLC_3D_Size (none) -> 2.2 2.2

Commit message: Updated the wiring for the 5V line to be connected to the +4V net. That is what it is named even though it is 4.5 ish volts.
Parts:
- AL1, AL2, AL3, AL4, AL5, AL6, AL7: JLC_3DModel_Q c6c295f7aed14366abe0e80218141640 -> (none); JLC_3D_Size 2.2 2.2 -> (none); LCSC Part C22371528 -> (none); Supplier Part (none) -> C22371528
- AL10, AL11, AL12, AL13, AL14, AL15, AL16, AL17, AL18, AL19, AL20, AL21, AL22, AL23, AL8, AL9: JLC_3DModel_Q c6c295f7aed14366abe0e80218141640 -> (none); JLC_3D_Size 2.2 2.2 -> (none)
