File: hardware/badge-esp32-s3/JST-PH.kicad_sch (KiCad schematic)
At the start: 1 part, among them CN1 B4B-PH-SM4-TB (LF)(SN)

Commit message: Spelling error correction
Other:
- note added: "Through Hole Component! Order Seperately!"
- note removed: "Through Hole Component!! Order Sepretly!"
Changed lines of the file:
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@@
 	(generator_version "9.0")
 	(paper "A4")
-	(text "Through Hole Component!! Order Sepretly! "
+	(text "Through Hole Component! Order Seperately! "
 		(exclude_from_sim no)
 		(at 148.59 57.15 0)
