File: hardware/badge-esp32-s3/usbc_5v_v2_data.kicad_sch (KiCad schematic)
At the start: 8 parts, among them J1 Connector, USB-TYPE-C-16P

Commit message: Annotate schematic
Parts:
- renumbered C7 to C5, D3 to D2, D4 to D3, D2 to D4, D1 to D5
Changed lines of the file:
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@@
 		(on_board yes)
 		(dnp no)
-		(property "Reference" "#PWR03"
+		(property "Reference" "#PWR011"
 			(at 138.43 68.58 0)
 			(effects
@@
 			(project "badge-esp32-s3"
 				(path "/e2af9a6c-dbe9-4de2-9ba6-ea213a7300ec/791664b9-b2ed-4f3b-9466-1f499155c51d"
+					(reference "#PWR018")
+					(unit 1)
+				)
+				(path "/e2af9a6c-dbe9-4de2-9ba6-ea213a7300ec/e365f6ed-f2b4-4ac9-8336-75c01e8e2e23"
 					(reference "#PWR011")
-					(unit 1)
-				)
-				(path "/e2af9a6c-dbe9-4de2-9ba6-ea213a7300ec/e365f6ed-f2b4-4ac9-8336-75c01e8e2e23"
-					(reference "#PWR03")
 					(unit 1)
 				)
@@
 		(on_board yes)
 		(dnp no)
-		(property "Reference" "D2"
+		(property "Reference" "D4"
 			(at 152.654 67.564 90)
 			(effects
@@
 			(project "badge-esp32-s3"
 				(path "/e2af9a6c-dbe9-4de2-9ba6-ea213a7300ec/791664b9-b2ed-4f3b-9466-1f499155c51d"
-					(reference "D7")
+					(reference "D8")
 					(unit 1)
 				)
 				(path "/e2af9a6c-dbe9-4de2-9ba6-ea213a7300ec/e365f6ed-f2b4-4ac9-8336-75c01e8e2e23"
-					(reference "D2")
+					(reference "D4")
 					(unit 1)
 				)
@@
 		(dnp no)
 		(fields_autoplaced yes)
-		(property "Reference" "#PWR07"
+		(property "Reference" "#PWR010"
 			(at 129.54 116.84 0)
 			(effects
@@
 			(project "badge-esp32-s3"
 				(path "/e2af9a6c-dbe9-4de2-9ba6-ea213a7300ec/791664b9-b2ed-4f3b-9466-1f499155c51d"
+					(reference "#PWR017")
+					(unit 1)
+				)
+				(path "/e2af9a6c-dbe9-4de2-9ba6-ea213a7300ec/e365f6ed-f2b4-4ac9-8336-75c01e8e2e23"
 					(reference "#PWR010")
-					(unit 1)
-				)
-				(path "/e2af9a6c-dbe9-4de2-9ba6-ea213a7300ec/e365f6ed-f2b4-4ac9-8336-75c01e8e2e23"
-					(reference "#PWR07")
 					(unit 1)
 				)
@@
 		(dnp no)
 		(fields_autoplaced yes)
-		(property "Reference" "#PWR02"
+		(property "Reference" "#PWR09"
 			(at 109.22 105.41 0)
 			(effects
@@
 			(project "badge-esp32-s3"
 				(path "/e2af9a6c-dbe9-4de2-9ba6-ea213a7300ec/791664b9-b2ed-4f3b-9466-1f499155c51d"
+					(reference "#PWR016")
+					(unit 1)
+				)
+				(path "/e2af9a6c-dbe9-4de2-9ba6-ea213a7300ec/e365f6ed-f2b4-4ac9-8336-75c01e8e2e23"
 					(reference "#PWR09")
-					(unit 1)
-				)
-				(path "/e2af9a6c-dbe9-4de2-9ba6-ea213a7300ec/e365f6ed-f2b4-4ac9-8336-75c01e8e2e23"
-					(reference "#PWR02")
 					(unit 1)
 				)
@@
 		(dnp no)
 		(fields_autoplaced yes)
-		(property "Reference" "D1"
+		(property "Reference" "D5"
 			(at 159.0675 54.61 90)
 			(effects
@@
 			(project ""
 				(path "/e2af9a6c-dbe9-4de2-9ba6-ea213a7300ec/791664b9-b2ed-4f3b-9466-1f499155c51d"
-					(reference "D8")
+					(reference "D9")
 					(unit 1)
 				)
 				(path "/e2af9a6c-dbe9-4de2-9ba6-ea213a7300ec/e365f6ed-f2b4-4ac9-8336-75c01e8e2e23"
-					(reference "D1")
+					(reference "D5")
 					(unit 1)
 				)
@@
 		(on_board yes)
 		(dnp no)
-		(property "Reference" "D4"
+		(property "Reference" "D3"
 			(at 146.05 92.7099 90)
 			(effects
@@
 			(project "badge-esp32-s3"
 				(path "/e2af9a6c-dbe9-4de2-9ba6-ea213a7300ec/791664b9-b2ed-4f3b-9466-1f499155c51d"
-					(reference "D6")
+					(reference "D7")
 					(unit 1)
 				)
 				(path "/e2af9a6c-dbe9-4de2-9ba6-ea213a7300ec/e365f6ed-f2b4-4ac9-8336-75c01e8e2e23"
-					(reference "D4")
+					(reference "D3")
 					(unit 1)
 				)
@@
 		(dnp no)
 		(fields_autoplaced yes)
-		(property "Reference" "#PWR04"
+		(property "Reference" "#PWR013"
 			(at 151.13 82.55 0)
 			(effects
@@
 			(project "badge-esp32-s3"
 				(path "/e2af9a6c-dbe9-4de2-9ba6-ea213a7300ec/791664b9-b2ed-4f3b-9466-1f499155c51d"
+					(reference "#PWR020")
+					(unit 1)
+				)
+				(path "/e2af9a6c-dbe9-4de2-9ba6-ea213a7300ec/e365f6ed-f2b4-4ac9-8336-75c01e8e2e23"
 					(reference "#PWR013")
-					(unit 1)
-				)
-				(path "/e2af9a6c-dbe9-4de2-9ba6-ea213a7300ec/e365f6ed-f2b4-4ac9-8336-75c01e8e2e23"
-					(reference "#PWR04")
 					(unit 1)
 				)
@@
 		(dnp no)
 		(fields_autoplaced yes)
-		(property "Reference" "#PWR06"
+		(property "Reference" "#PWR012"
 			(at 142.24 116.84 0)
 			(effects
@@
 			(project "badge-esp32-s3"
 				(path "/e2af9a6c-dbe9-4de2-9ba6-ea213a7300ec/791664b9-b2ed-4f3b-9466-1f499155c51d"
+					(reference "#PWR019")
+					(unit 1)
+				)
+				(path "/e2af9a6c-dbe9-4de2-9ba6-ea213a7300ec/e365f6ed-f2b4-4ac9-8336-75c01e8e2e23"
 					(reference "#PWR012")
-					(unit 1)
-				)
-				(path "/e2af9a6c-dbe9-4de2-9ba6-ea213a7300ec/e365f6ed-f2b4-4ac9-8336-75c01e8e2e23"
-					(reference "#PWR06")
 					(unit 1)
 				)
@@
 		(on_board yes)
 		(dnp no)
-		(property "Reference" "D3"
+		(property "Reference" "D2"
 			(at 133.35 93.9799 90)
 			(effects
@@
 			(project "badge-esp32-s3"
 				(path "/e2af9a6c-dbe9-4de2-9ba6-ea213a7300ec/791664b9-b2ed-4f3b-9466-1f499155c51d"
-					(reference "D5")
+					(reference "D6")
 					(unit 1)
 				)
 				(path "/e2af9a6c-dbe9-4de2-9ba6-ea213a7300ec/e365f6ed-f2b4-4ac9-8336-75c01e8e2e23"
-					(reference "D3")
+					(reference "D2")
 					(unit 1)
 				)
@@
 		(dnp no)
 		(fields_autoplaced yes)
-		(property "Reference" "C7"
+		(property "Reference" "C5"
 			(at 168.91 64.7699 0)
 			(effects
@@
 			(project "badge-esp32-s3"
 				(path "/e2af9a6c-dbe9-4de2-9ba6-ea213a7300ec/791664b9-b2ed-4f3b-9466-1f499155c51d"
-					(reference "C8")
+					(reference "C6")
 					(unit 1)
 				)
 				(path "/e2af9a6c-dbe9-4de2-9ba6-ea213a7300ec/e365f6ed-f2b4-4ac9-8336-75c01e8e2e23"
-					(reference "C7")
+					(reference "C5")
 					(unit 1)
 				)
@@
 		(dnp no)
 		(fields_autoplaced yes)
-		(property "Reference" "#PWR01"
+		(property "Reference" "#PWR08"
 			(at 101.6 105.41 0)
 			(effects
@@
 			(project "badge-esp32-s3"
 				(path "/e2af9a6c-dbe9-4de2-9ba6-ea213a7300ec/791664b9-b2ed-4f3b-9466-1f499155c51d"
+					(reference "#PWR015")
+					(unit 1)
+				)
+				(path "/e2af9a6c-dbe9-4de2-9ba6-ea213a7300ec/e365f6ed-f2b4-4ac9-8336-75c01e8e2e23"
 					(reference "#PWR08")
-					(unit 1)
-				)
-				(path "/e2af9a6c-dbe9-4de2-9ba6-ea213a7300ec/e365f6ed-f2b4-4ac9-8336-75c01e8e2e23"
-					(reference "#PWR01")
 					(unit 1)
 				)
@@
 		(dnp no)
 		(fields_autoplaced yes)
-		(property "Reference" "#PWR05"
+		(property "Reference" "#PWR014"
 			(at 166.37 80.01 0)
 			(effects
@@
 			(project "badge-esp32-s3"
 				(path "/e2af9a6c-dbe9-4de2-9ba6-ea213a7300ec/791664b9-b2ed-4f3b-9466-1f499155c51d"
+					(reference "#PWR021")
+					(unit 1)
+				)
+				(path "/e2af9a6c-dbe9-4de2-9ba6-ea213a7300ec/e365f6ed-f2b4-4ac9-8336-75c01e8e2e23"
 					(reference "#PWR014")
 					(unit 1)
 				)
-				(path "/e2af9a6c-dbe9-4de2-9ba6-ea213a7300ec/e365f6ed-f2b4-4ac9-8336-75c01e8e2e23"
-					(reference "#PWR05")
-					(unit 1)
-				)
