File: hardware/badge-esp32-s3/minibadge.kicad_sch (KiCad schematic)
At the start: 15 parts, among them J12 Conn_01x02_Socket, J13 Conn_01x04_Socket, J5 Conn_01x02_Socket, J6 Conn_01x04_Socket, J7 Conn_01x08_Socket, J8 Conn_01x08_Socket, J9 Conn_02x06_Odd_Even

Commit message: finished component alignment
Parts:
- J12, J13, J5, J6, J9: FT Rotation Offset (none) -> -90
- J7, J8: FT Rotation Offset (none) -> -90; LCSC C42431862 -> C42385698
Changed lines of the file:
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@@
 			)
 		)
-		(property "LCSC" "C42431862"
+		(property "LCSC" "C42385698"
+			(at 102.87 67.31 0)
+			(effects
+				(font
+					(size 1.27 1.27)
+				)
+				(hide yes)
+			)
+		)
+		(property "FT Rotation Offset" "-90"
 			(at 102.87 67.31 0)
 			(effects
@@
 			)
 		)
+		(property "FT Rotation Offset" "-90"
+			(at 88.9 152.4 0)
+			(effects
+				(font
+					(size 1.27 1.27)
+				)
+				(hide yes)
+			)
+		)
 		(pin "11"
 		)
@@
 			)
 		)
+		(property "FT Rotation Offset" "-90"
+			(at 107.95 82.55 0)
+			(effects
+				(font
+					(size 1.27 1.27)
+				)
+				(hide yes)
+			)
+		)
 		(pin "1"
 		)
@@
 		)
 		(property "LCSC" "C7499322"
+			(at 152.4 82.55 0)
+			(effects
+				(font
+					(size 1.27 1.27)
+				)
+				(hide yes)
+			)
+		)
+		(property "FT Rotation Offset" "-90"
 			(at 152.4 82.55 0)
 			(effects
@@
 			)
 		)
-		(property "LCSC" "C42431862"
+		(property "LCSC" "C42385698"
+			(at 160.02 67.31 0)
+			(effects
+				(font
+					(size 1.27 1.27)
+				)
+				(hide yes)
+			)
+		)
+		(property "FT Rotation Offset" "-90"
 			(at 160.02 67.31 0)
 			(effects
@@
 			)
 		)
+		(property "FT Rotation Offset" "-90"
+			(at 95.25 82.55 0)
+			(effects
+				(font
+					(size 1.27 1.27)
+				)
+				(hide yes)
+			)
+		)
 		(pin "1"
 		)
@@
 			(at 165.1 82.55 0)
 			(effects
+				(font
+					(size 1.27 1.27)
+				)
+				(hide yes)
+			)
+		)
+		(property "FT Rotation Offset" "-90"
+			(at 165.1 82.55 0)
+			(effects
