File: hardware/badge-esp32-s3/exposed_pins.kicad_sch (KiCad schematic)
At the start: 8 parts, among them CN1 B4B-PH-SM4-TB (LF)(SN), CN3 HDR-TH_2P-P2.54-V-F, U19 FH2.54-09-02PZD, U6 ZX-SH1.0-4PWT

Commit message: Updated the wiring for the 5V line to be connected to the +4V net. That is what it is named even though it is 4.5 ish volts.
Parts:
- CN3: JLC_3DModel_Q 925d5dffa823422895d76d9dc6f5e8cd -> (none); JLC_3D_Size 5.48 2.5 -> (none)
- H2: JLC_3DModel_Q 412102dbb0884df38b5dec3a90c03673 -> (none); JLC_3D_Size 23.26 5 -> (none); LCSC Part C132125 -> (none); Supplier Part (none) -> C132125
- U14: JLC_3DModel_Q 14c20a80002e418c9c9633718d8bc2dd -> (none); JLC_3D_Size 7.62 5.01 -> (none)
Changed lines of the file:
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@@
-			)
-		)
-		(property "JLC_3DModel_Q" "925d5dffa823422895d76d9dc6f5e8cd"
-			(at 226.06 90.17 0)
-			(effects
-				(font
-					(size 1.27 1.27)
-				)
-				(hide yes)
-			)
-		)
-		(property "JLC_3D_Size" "5.48 2.5"
-			(at 226.06 90.17 0)
-			(effects
-				(font
-					(size 1.27 1.27)
-				)
-				(hide yes)
 			)
 		)
@@
 			)
 		)
+		(property "Supplier Part" "C132125"
+			(at 149.86 102.87 0)
+			(effects
+				(font
+					(size 1.27 1.27)
+				)
+				(hide yes)
+			)
+		)
 		(property "Supplier" "LCSC"
 			(at 149.86 102.87 0)
@@
 		)
 		(property "LCSC Part Name" "2x9P 间距:2.54mm 直插"
-			(at 149.86 102.87 0)
-			(effects
-				(font
-					(size 1.27 1.27)
-				)
-				(hide yes)
-			)
-		)
-		(property "JLC_3DModel_Q" "412102dbb0884df38b5dec3a90c03673"
-			(at 149.86 102.87 0)
-			(effects
-				(font
-					(size 1.27 1.27)
-				)
-				(hide yes)
-			)
-		)
-		(property "JLC_3D_Size" "23.26 5"
-			(at 149.86 102.87 0)
-			(effects
-				(font
-					(size 1.27 1.27)
-				)
-				(hide yes)
-			)
-		)
-		(property "LCSC Part" "C132125"
 			(at 149.86 102.87 0)
 			(effects
@@
 			(at 140.97 40.64 0)
 			(effects
-				(font
-					(size 1.27 1.27)
-				)
-				(hide yes)
-			)
-		)
-		(property "JLC_3DModel_Q" "14c20a80002e418c9c9633718d8bc2dd"
-			(at 140.97 40.64 0)
-			(effects
-				(font
-					(size 1.27 1.27)
-				)
-				(hide yes)
-			)
-		)
-		(property "JLC_3D_Size" "7.62 5.01"
-			(at 140.97 40.64 0)
-			(effects

Commit message: minibadge_fix?
Parts:
- CN3: JLC_3DModel_Q (none) -> 925d5dffa823422895d76d9dc6f5e8cd; JLC_3D_Size (none) -> 5.48 2.5
- H2: JLC_3DModel_Q (none) -> 412102dbb0884df38b5dec3a90c03673; JLC_3D_Size (none) -> 23.26 5; LCSC Part (none) -> C132125; Supplier Part C132125 -> (none)
- U14: JLC_3DModel_Q (none) -> 14c20a80002e418c9c9633718d8bc2dd; JLC_3D_Size (none) -> 7.62 5.01
Changed lines of the file:
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@@
+			)
+		)
+		(property "JLC_3DModel_Q" "925d5dffa823422895d76d9dc6f5e8cd"
+			(at 226.06 90.17 0)
+			(effects
+				(font
+					(size 1.27 1.27)
+				)
+				(hide yes)
+			)
+		)
+		(property "JLC_3D_Size" "5.48 2.5"
+			(at 226.06 90.17 0)
+			(effects
+				(font
+					(size 1.27 1.27)
+				)
+				(hide yes)
 			)
 		)
@@
 			)
 		)
-		(property "Supplier Part" "C132125"
-			(at 149.86 102.87 0)
-			(effects
-				(font
-					(size 1.27 1.27)
-				)
-				(hide yes)
-			)
-		)
 		(property "Supplier" "LCSC"
 			(at 149.86 102.87 0)
@@
 		)
 		(property "LCSC Part Name" "2x9P 间距:2.54mm 直插"
+			(at 149.86 102.87 0)
+			(effects
+				(font
+					(size 1.27 1.27)
+				)
+				(hide yes)
+			)
+		)
+		(property "JLC_3DModel_Q" "412102dbb0884df38b5dec3a90c03673"
+			(at 149.86 102.87 0)
+			(effects
+				(font
+					(size 1.27 1.27)
+				)
+				(hide yes)
+			)
+		)
+		(property "JLC_3D_Size" "23.26 5"
+			(at 149.86 102.87 0)
+			(effects
+				(font
+					(size 1.27 1.27)
+				)
+				(hide yes)
+			)
+		)
+		(property "LCSC Part" "C132125"
 			(at 149.86 102.87 0)
 			(effects
@@
 			(at 140.97 40.64 0)
 			(effects
+				(font
+					(size 1.27 1.27)
+				)
+				(hide yes)
+			)
+		)
+		(property "JLC_3DModel_Q" "14c20a80002e418c9c9633718d8bc2dd"
+			(at 140.97 40.64 0)
+			(effects
+				(font
+					(size 1.27 1.27)
+				)
+				(hide yes)
+			)
+		)
+		(property "JLC_3D_Size" "7.62 5.01"
+			(at 140.97 40.64 0)
+			(effects
