File: hardware/badge-esp32-s3/gpio_header_block.kicad_sch (KiCad schematic)
At the start: 1 part, among them U20 2x14_female

Commit message: minibadge_fix?
Parts:
- U20: JLC_3DModel_Q (none) -> 3b7fbf5db20b4c58b7d710ca6a34c9ed; JLC_3D_Size (none) -> 36.06 5; LCSC Part (none) -> C42372538; Supplier Part C42372538 -> (none)
Changed lines of the file:
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@@
-			)
-		)
-		(property "Supplier Part" "C42372538"
-			(at 129.54 91.44 0)
-			(effects
-				(font
-					(size 1.27 1.27)
-				)
-				(hide yes)
 			)
 		)
@@
 			(at 129.54 91.44 0)
 			(effects
+				(font
+					(size 1.27 1.27)
+				)
+				(hide yes)
+			)
+		)
+		(property "JLC_3DModel_Q" "3b7fbf5db20b4c58b7d710ca6a34c9ed"
+			(at 129.54 91.44 0)
+			(effects
+				(font
+					(size 1.27 1.27)
+				)
+				(hide yes)
+			)
+		)
+		(property "JLC_3D_Size" "36.06 5"
+			(at 129.54 91.44 0)
+			(effects
+				(font
+					(size 1.27 1.27)
+				)
+				(hide yes)
+			)
+		)
+		(property "LCSC Part" "C42372538"
+			(at 129.54 91.44 0)
+			(effects

Commit message: Updated the wiring for the 5V line to be connected to the +4V net. That is what it is named even though it is 4.5 ish volts.
Parts:
- U20: JLC_3DModel_Q 3b7fbf5db20b4c58b7d710ca6a34c9ed -> (none); JLC_3D_Size 36.06 5 -> (none); LCSC Part C42372538 -> (none); Supplier Part (none) -> C42372538
Changed lines of the file:
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@@
+			)
+		)
+		(property "Supplier Part" "C42372538"
+			(at 129.54 91.44 0)
+			(effects
+				(font
+					(size 1.27 1.27)
+				)
+				(hide yes)
 			)
 		)
@@
 			(at 129.54 91.44 0)
 			(effects
-				(font
-					(size 1.27 1.27)
-				)
-				(hide yes)
-			)
-		)
-		(property "JLC_3DModel_Q" "3b7fbf5db20b4c58b7d710ca6a34c9ed"
-			(at 129.54 91.44 0)
-			(effects
-				(font
-					(size 1.27 1.27)
-				)
-				(hide yes)
-			)
-		)
-		(property "JLC_3D_Size" "36.06 5"
-			(at 129.54 91.44 0)
-			(effects
-				(font
-					(size 1.27 1.27)
-				)
-				(hide yes)
-			)
-		)
-		(property "LCSC Part" "C42372538"
-			(at 129.54 91.44 0)
-			(effects
