File: hardware/badge-esp32-s3/Accelormeter.kicad_sch (KiCad schematic)
At the start: 6 parts, among them U1 MMA8452QR1_C11360

Commit message: Annotate schematic
Parts:
- renumbered C20 to C24, C21 to C25, C22 to C26, R30 to R39, R29 to R40, U1 to U18
Changed lines of the file:
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@@
 		(dnp no)
 		(fields_autoplaced yes)
-		(property "Reference" "R30"
+		(property "Reference" "R39"
 			(at 102.87 74.9299 0)
 			(effects
@@
 			(project ""
 				(path "/e2af9a6c-dbe9-4de2-9ba6-ea213a7300ec/9feb22ac-0492-47b5-89fe-3e77a54de168/ed10a1a3-8649-458b-a567-b8a974afd909"
-					(reference "R30")
+					(reference "R39")
 					(unit 1)
 				)
@@
 		(dnp no)
 		(fields_autoplaced yes)
-		(property "Reference" "#PWR044"
+		(property "Reference" "#PWR061"
 			(at 165.1 85.09 0)
 			(effects
@@
 			(project ""
 				(path "/e2af9a6c-dbe9-4de2-9ba6-ea213a7300ec/9feb22ac-0492-47b5-89fe-3e77a54de168/ed10a1a3-8649-458b-a567-b8a974afd909"
-					(reference "#PWR044")
+					(reference "#PWR061")
 					(unit 1)
 				)
@@
 		(dnp no)
 		(fields_autoplaced yes)
-		(property "Reference" "C21"
+		(property "Reference" "C25"
 			(at 109.22 62.2301 0)
 			(effects
@@
 			(project ""
 				(path "/e2af9a6c-dbe9-4de2-9ba6-ea213a7300ec/9feb22ac-0492-47b5-89fe-3e77a54de168/ed10a1a3-8649-458b-a567-b8a974afd909"
-					(reference "C21")
+					(reference "C25")
 					(unit 1)
 				)
@@
 		(dnp no)
 		(fields_autoplaced yes)
-		(property "Reference" "#PWR045"
+		(property "Reference" "#PWR059"
 			(at 124.46 78.74 0)
 			(effects
@@
 			(project ""
 				(path "/e2af9a6c-dbe9-4de2-9ba6-ea213a7300ec/9feb22ac-0492-47b5-89fe-3e77a54de168/ed10a1a3-8649-458b-a567-b8a974afd909"
-					(reference "#PWR045")
+					(reference "#PWR059")
 					(unit 1)
 				)
@@
 		(dnp no)
 		(fields_autoplaced yes)
-		(property "Reference" "#PWR015"
+		(property "Reference" "#PWR060"
 			(at 123.19 80.01 0)
 			(effects
@@
 			(project ""
 				(path "/e2af9a6c-dbe9-4de2-9ba6-ea213a7300ec/9feb22ac-0492-47b5-89fe-3e77a54de168/ed10a1a3-8649-458b-a567-b8a974afd909"
-					(reference "#PWR015")
+					(reference "#PWR060")
 					(unit 1)
 				)
@@
 		(dnp no)
 		(fields_autoplaced yes)
-		(property "Reference" "R29"
+		(property "Reference" "R40"
 			(at 113.03 74.9299 0)
 			(effects
@@
 			(project ""
 				(path "/e2af9a6c-dbe9-4de2-9ba6-ea213a7300ec/9feb22ac-0492-47b5-89fe-3e77a54de168/ed10a1a3-8649-458b-a567-b8a974afd909"
-					(reference "R29")
+					(reference "R40")
 					(unit 1)
 				)
@@
 		(dnp no)
 		(fields_autoplaced yes)
-		(property "Reference" "C22"
+		(property "Reference" "C26"
 			(at 167.64 71.1199 0)
 			(effects
@@
 			(project ""
 				(path "/e2af9a6c-dbe9-4de2-9ba6-ea213a7300ec/9feb22ac-0492-47b5-89fe-3e77a54de168/ed10a1a3-8649-458b-a567-b8a974afd909"
-					(reference "C22")
+					(reference "C26")
 					(unit 1)
 				)
@@
 		(dnp no)
 		(fields_autoplaced yes)
-		(property "Reference" "U1"
+		(property "Reference" "U18"
 			(at 143.51 62.23 0)
 			(effects
@@
 			(project ""
 				(path "/e2af9a6c-dbe9-4de2-9ba6-ea213a7300ec/9feb22ac-0492-47b5-89fe-3e77a54de168/ed10a1a3-8649-458b-a567-b8a974afd909"
-					(reference "U1")
+					(reference "U18")
 					(unit 1)
 				)
@@
 		(dnp no)
 		(fields_autoplaced yes)
-		(property "Reference" "C20"
+		(property "Reference" "C24"
 			(at 101.6 62.2301 0)
 			(effects
@@
 			(project ""
 				(path "/e2af9a6c-dbe9-4de2-9ba6-ea213a7300ec/9feb22ac-0492-47b5-89fe-3e77a54de168/ed10a1a3-8649-458b-a567-b8a974afd909"
-					(reference "C20")
+					(reference "C24")
 					(unit 1)
 				)
@@
 		(dnp no)
 		(fields_autoplaced yes)
-		(property "Reference" "#PWR016"
+		(property "Reference" "#PWR062"
 			(at 175.26 80.01 0)
 			(effects
@@
 			(project ""
 				(path "/e2af9a6c-dbe9-4de2-9ba6-ea213a7300ec/9feb22ac-0492-47b5-89fe-3e77a54de168/ed10a1a3-8649-458b-a567-b8a974afd909"
-					(reference "#PWR016")
+					(reference "#PWR062")
 					(unit 1)
 				)

Commit message: Fix some DRC errors
Connections:
- no-connect marks 0 -> 5
Changed lines of the file:
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@@
 		(color 0 0 0 0)
+	)
+	(no_connect
+		(at 154.94 77.47)
+	)
+	(no_connect
+		(at 132.08 87.63)
+	)
+	(no_connect
+		(at 154.94 72.39)
+	)
+	(no_connect
+		(at 132.08 74.93)
+	)
+	(no_connect
+		(at 154.94 69.85)
 	)
 	(wire

Commit message: almost finished
Parts:
- removed C24, C25: 100nF, PCM_JLCPCB:C_0603, symbol PCM_JLCPCB-Capacitors:0603,100nF
- removed R39, R40: 4.7kΩ, PCM_JLCPCB:R_0603, symbol PCM_JLCPCB-Resistors:0603,4.7kΩ
- added C10, C11: 100nF, PCM_JLCPCB:C_0402, symbol PCM_JLCPCB-Capacitors:0402,100nF
- added R43, R45: 4.7kΩ, PCM_JLCPCB:R_0402, symbol PCM_JLCPCB-Resistors:0402,4.7kΩ
Connections:
- net 3.3v in: now also C10.1, R43.1, R45.1
- net GND: now also C10.2, C11.2
- net SCL: now also R43.2
- net SDA: now also R45.2
- net at U18.2 (BYP): now also C11.1
