File: hardware/badge-esp32-s3/Charging.kicad_sch (KiCad schematic)
At the start: 11 parts, among them P1 PH-2A_C2319, Q3 HL2301A, U4 TP4056

Commit message: almost finished
Parts:
- added Q6: AO3424, lcsc-lib:SC-59-3_L2.9-W1.6-P0.95-LS2.9-BR, symbol lcsc-lib:AO3424
- added R48: 100kΩ, PCM_JLCPCB:R_0402, symbol PCM_JLCPCB-Resistors:0402,100kΩ
Connections:
- net GND: now also Q6.2 (S); no longer P1.2
- net VBATT: now also R48.2
- new net: Q6.1 (G), R48.1
- new net: P1.2, Q6.3 (D)
Other:
- moved on the sheet: P1
