File: hardware/badge-esp32-s3/onboard_peripheral.kicad_sch (KiCad schematic)
At the start: 1 part

Commit message: final changes and part updated
Parts:
- removed CN2: ~, lcsc-lib:HDR-TH_2P-P2.54-V-F, symbol lcsc-lib:HX PM2.54-1X2P ZC-Y
- added J15: Conn_01x02_Socket, Connector_PinSocket_2.54mm:PinSocket_1x02_P2.54mm_Vertical, symbol Connector:Conn_01x02_Socket
Connections:
- net Accelormeter/INT 1 (output to MCU, NN) : now also J15.2 (Pin_2)
- net Accelormeter/INT 2 (output to MCU, NN) : now also J15.1 (Pin_1)
Changed lines of the file:
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@@
 	)
 	(symbol
-		(lib_id "lcsc-lib:HX PM2.54-1X2P ZC-Y")
-		(at 26.67 154.94 180)
+		(lib_id "Connector:Conn_01x02_Socket")
+		(at 26.67 156.21 180)
 		(unit 1)
 		(exclude_from_sim no)
@@
 		(dnp no)
 		(fields_autoplaced yes)
-		(property "Reference" "CN2"
-			(at 26.67 146.05 0)
+		(property "Reference" "J15"
+			(at 27.305 148.59 0)
 			(effects
 				(font
@@
 			)
 		)
-		(property "Value" "~"
-			(at 26.67 148.59 0)
+		(property "Value" "Conn_01x02_Socket"
+			(at 27.305 151.13 0)
 			(effects
 				(font
@@
 			)
 		)
-		(property "Footprint" "lcsc-lib:HDR-TH_2P-P2.54-V-F"
-			(at 26.67 154.94 0)
+		(property "Footprint" "Connector_PinSocket_2.54mm:PinSocket_1x02_P2.54mm_Vertical"
+			(at 26.67 156.21 0)
 			(effects
 				(font
@@
 			)
 		)
-		(property "Datasheet" "https://item.szlcsc.com/datasheet/HX%2520PM2.54-1x2P%2520ZC-Y/24075299.html"
-			(at 26.67 154.94 0)
+		(property "Datasheet" "~"
+			(at 26.67 156.21 0)
 			(effects
 				(font
@@
 			)
 		)
-		(property "Description" "Holes Structure:1x2P Pitch:2.54mm Row Spacing:- Circular Hole / Square Hole:Square Hole Mounting Type:Through Hole Number of Rows:1 Number of Positions:2P Current Rating:3A Voltage Rating (Max):1kV Holes Direction:Top Insulation Height:8.5mm Contact Mater"
-			(at 26.67 154.94 0)
+		(property "Description" "Generic connector, single row, 01x02, script generated"
+			(at 26.67 156.21 0)
 			(effects
 				(font
@@
 			)
 		)
-		(property "Manufacturer Part" "HX PM2.54-1x2P ZC-Y"
-			(at 26.67 154.94 0)
+		(property "LCSC" "C7499322"
+			(at 26.67 156.21 0)
 			(effects
 				(font
@@
 			)
 		)
-		(property "Manufacturer" "hanxia(韩下)"
-			(at 26.67 154.94 0)
-			(effects
-				(font
-					(size 1.27 1.27)
-				)
-				(hide yes)
-			)
-		)
-		(property "Supplier Part" "C22438152"
-			(at 26.67 154.94 0)
-			(effects
-				(font
-					(size 1.27 1.27)
-				)
-				(hide yes)
-			)
-		)
-		(property "Supplier" "LCSC"
-			(at 26.67 154.94 0)
-			(effects
-				(font
-					(size 1.27 1.27)
-				)
-				(hide yes)
-			)
-		)
-		(property "LCSC Part Name" "1x2P 间距:2.54mm 直插"
-			(at 26.67 154.94 0)
-			(effects
-				(font
-					(size 1.27 1.27)
-				)
-				(hide yes)
-			)
+		(pin "2"
 		)
 		(pin "1"
 		)
-		(pin "2"
-		)
 		(instances
-			(project ""
+			(project "badge-esp32-s3"
 				(path "/e2af9a6c-dbe9-4de2-9ba6-ea213a7300ec/9feb22ac-0492-47b5-89fe-3e77a54de168"
-					(reference "CN2")
+					(reference "J15")
 					(unit 1)
 				)

Commit message: finished component alignment
Parts:
- J15: FT Rotation Offset (none) -> -90
Changed lines of the file:
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@@
+			)
+		)
+		(property "FT Rotation Offset" "-90"
+			(at 26.67 156.21 0)
+			(effects
+				(font
+					(size 1.27 1.27)
+				)
+				(hide yes)
 			)
 		)
