File: hardware/badge-esp32-s3/uart_interface.kicad_sch (KiCad schematic)
At the start: 17 parts, among them Q1 SS8050 200-350, Q2 SS8050 200-350, U3 CP2102N-A02-GQFN28R

Commit message: Annotate schematic
Parts:
- renumbered C9 to C7, C10 to C8, C11 to C9
Changed lines of the file:
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@@
 		(dnp no)
 		(fields_autoplaced yes)
-		(property "Reference" "C11"
+		(property "Reference" "C9"
 			(at 234.95 71.1199 0)
 			(effects
@@
 			(project ""
 				(path "/e2af9a6c-dbe9-4de2-9ba6-ea213a7300ec/94c82a22-114c-4c54-9d6a-9512e8cebb9e"
-					(reference "C11")
+					(reference "C9")
 					(unit 1)
 				)
@@
 		(dnp no)
 		(fields_autoplaced yes)
-		(property "Reference" "#PWR023"
+		(property "Reference" "#PWR022"
 			(at 34.29 107.95 0)
 			(effects
@@
 			(project ""
 				(path "/e2af9a6c-dbe9-4de2-9ba6-ea213a7300ec/94c82a22-114c-4c54-9d6a-9512e8cebb9e"
-					(reference "#PWR023")
+					(reference "#PWR022")
 					(unit 1)
 				)
@@
 		(dnp no)
 		(fields_autoplaced yes)
-		(property "Reference" "#PWR022"
+		(property "Reference" "#PWR025"
 			(at 60.96 81.28 0)
 			(effects
@@
 			(project ""
 				(path "/e2af9a6c-dbe9-4de2-9ba6-ea213a7300ec/94c82a22-114c-4c54-9d6a-9512e8cebb9e"
-					(reference "#PWR022")
+					(reference "#PWR025")
 					(unit 1)
 				)
@@
 		(dnp no)
 		(fields_autoplaced yes)
-		(property "Reference" "#PWR025"
+		(property "Reference" "#PWR024"
 			(at 63.5 137.16 0)
 			(effects
@@
 			(project ""
 				(path "/e2af9a6c-dbe9-4de2-9ba6-ea213a7300ec/94c82a22-114c-4c54-9d6a-9512e8cebb9e"
-					(reference "#PWR025")
+					(reference "#PWR024")
 					(unit 1)
 				)
@@
 		(dnp no)
 		(fields_autoplaced yes)
-		(property "Reference" "C9"
+		(property "Reference" "C7"
 			(at 36.83 92.7099 0)
 			(effects
@@
 			(project ""
 				(path "/e2af9a6c-dbe9-4de2-9ba6-ea213a7300ec/94c82a22-114c-4c54-9d6a-9512e8cebb9e"
-					(reference "C9")
+					(reference "C7")
 					(unit 1)
 				)
@@
 		(dnp no)
 		(fields_autoplaced yes)
-		(property "Reference" "C10"
+		(property "Reference" "C8"
 			(at 49.53 116.8399 0)
 			(effects
@@
 			(project ""
 				(path "/e2af9a6c-dbe9-4de2-9ba6-ea213a7300ec/94c82a22-114c-4c54-9d6a-9512e8cebb9e"
-					(reference "C10")
+					(reference "C8")
 					(unit 1)
 				)
@@
 		(dnp no)
 		(fields_autoplaced yes)
-		(property "Reference" "#PWR024"
+		(property "Reference" "#PWR023"
 			(at 34.29 134.62 0)
 			(effects
@@
 			(project ""
 				(path "/e2af9a6c-dbe9-4de2-9ba6-ea213a7300ec/94c82a22-114c-4c54-9d6a-9512e8cebb9e"
-					(reference "#PWR024")
+					(reference "#PWR023")
 					(unit 1)
 				)

Commit message: almost finished
Parts:
- removed R15, R16: 0Ω, PCM_JLCPCB:R_0402, symbol PCM_JLCPCB-Resistors:0402,0Ω
- added R15, R16: 470Ω, PCM_JLCPCB:R_0402, symbol PCM_JLCPCB-Resistors:0402,470Ω
Connections:
- net ENABLE: now also R15.2
- net MODE: now also R16.2
- net at Q1.3 (C): now also R15.1
- net at Q2.3 (C): now also R16.1
