File: hardware/badge-esp32-s3/display.kicad_sch (KiCad schematic)
At the start: 2 parts, among them P2 FPC 0.5MM 12P Pull type H2.0m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

Commit message: almost finished
Parts:
- added TP1, TP2, TP3, TP4, TP5: TestPoint, TestPoint:TestPoint_Pad_D1.5mm, symbol Connector:TestPoint
- added U7: HS20HS072RX-fpc, lcsc-lib:OLED-SMD_HS20HS072RX-pins_removed, symbol lcsc-lib:HS20HS072RX-fpc
Connections:
- net CS: now also TP1.1
- net D/C: now also TP2.1
- net RST: now also TP5.1
- net SCL: now also TP3.1
- net SDA: now also TP4.1

Commit message: final changes and part updated
Parts:
- added R39: 100kΩ, PCM_JLCPCB:R_0402, symbol PCM_JLCPCB-Resistors:0402,100kΩ
Connections:
- net GND: now also R39.2
- net RST: now also R39.1
Other:
- note added: "Default: Reset State"
