File: hardware/badge-esp32-s3/display.kicad_sch (KiCad schematic)
At the start: 9 parts, among them P2 FPC 0.5MM 12P Pull type H2.0m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, U7 HS20HS072RX-fpc

Commit message: changed buck/boost reg and final touchups
Parts:
- U7: now left out of the parts list
Changed lines of the file:
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@@
 		(unit 1)
 		(exclude_from_sim no)
-		(in_bom yes)
+		(in_bom no)
 		(on_board yes)
 		(dnp no)
